File: pcb/left/left.kicad_pcb (KiCad board)
At the start: 2 copper layers, 163.5 x 132.8 mm, 66 parts

Commit message: Redid left routing
Parts:
- moved D9 85.3 mm to (172.9, 133.0)
- moved S17 85.3 mm to (210.9, 128.0)
- moved H1 85.3 mm to (163.4, 99.5)
- moved D10 85.3 mm to (172.9, 114.0)
- moved S18 85.3 mm to (210.9, 109.0)
- moved D6 85.3 mm to (151.6, 121.1)
- moved S14 85.3 mm to (191.9, 106.0)
- moved H4 85.3 mm to (220.4, 139.0)
- moved D18 85.3 mm to (210.9, 114.0)
- moved S25 85.3 mm to (220.4, 172.7)
- moved S21 85.3 mm to (229.9, 131.0)
- moved D13 85.3 mm to (191.9, 130.0)
- moved H3 85.3 mm to (220.4, 101.0)
- moved S4 85.3 mm to (153.3, 154.0)
- moved D5 85.3 mm to (152.6, 140.1)
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Routing:
- net col1: track 246.7 -> 254.8 mm
- net col2: track 222.1 -> 228.2 mm
- net RE_A: track 67.3 -> 71.2 mm, vias 1 -> 0
- net col6: track 160.8 -> 163.2 mm
- net col3: track 196.3 -> 198.0 mm
- net VCC: track 30.3 -> 28.9 mm
- net col4: track 168.9 -> 170.3 mm
- net col7: track 162.9 -> 164.2 mm
- net RE_C: track 91.4 -> 92.4 mm
- net row1: track 131.7 -> 132.6 mm
- net row4: track 236.2 -> 235.3 mm
- net row2: track 172.2 -> 173.1 mm
- net row5: track 135.6 -> 136.4 mm
- net RAW: track 28.6 -> 27.8 mm
- net SCL: track 26.1 -> 25.3 mm
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Other:
- board text added: "L"
- board text added: "Rev1 github.com/mroetsc/krypton-kbd"
